Commit message: Included camera sensors in the simulation

File: paquetes_simulacion/rb1_base_description/robots/robotDummy.urdf (robot description, URDF)
Before this commit: robot rb1_base, 69 links, 68 joints
Links:
- added link camera_link
- added link joint_support_link
- added link rgbd_link
- added link shoulder_link
- added link support_end_link
Joints:
- added joint rb1_to_shoulder: type fixed, parent rb1_base_footprint, child shoulder_link, origin xyz=0.007 0 1.254 rpy=0 0 0
- added joint rgbd_to_camera: type fixed, parent rgbd_link, child camera_link, origin xyz=0 0 0 rpy=0 0 3.141592
- added joint shoulder_to_support_joint: type fixed, parent shoulder_link, child joint_support_link, origin xyz=0.115 0 0.030 rpy=0 0.785398 0
- added joint support_end_to_rgbd: type fixed, parent support_end_link, child rgbd_link, origin xyz=0.01803 0.0175 0 rpy=-1.5708 0 -1.5708
- added joint support_joint_to_end: type fixed, parent joint_support_link, child support_end_link, origin xyz=0.027 0 0.0425 rpy=0 0 0

Commit message: Moving camera

File: paquetes_simulacion/rb1_base_description/robots/robotDummy.urdf (robot description, URDF)
Before this commit: robot rb1_base, 74 links, 73 joints
Joints:
- joint shoulder_to_support_joint: axis (none) -> 0 -1 0; limit (none) -> lower=0 upper=1.5708 effort=50 velocity=1; type fixed -> revolute

Commit message: Camera meshes and hands_kinematics update

File: paquetes_simulacion/rb1_base_description/robots/robotDummy.urdf (robot description, URDF)
Before this commit: robot rb1_base, 74 links, 73 joints
Links:
- link camera_link: geometry visual mesh filename=package://rb1_base_description/meshes/others/D435i_Solid.stl scale=0.001 0.001 0.001
- link joint_support_link: geometry visual mesh filename=package://rb1_base_description/meshes/others/camera_support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 scale=0.0254 0.0254 0.0254
- link shoulder_link: geometry visual mesh filename=package://rb1_base_description/meshes/others/camera_support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 scale=0.0254 0.0254 0.0254
- link support_end_link: geometry visual mesh filename=package://rb1_base_description/meshes/others/camera_support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 scale=0.0254 0.0254 0.0254

Commit message: Collisions fixed and urdf file updated

File: paquetes_simulacion/rb1_base_description/robots/robotDummy.urdf (robot description, URDF)
Before this commit: robot rb1_base, 74 links, 73 joints
Links:
- link rb1_base_link: mass 25.0 -> 100.0
- link rb1_left_wheel_link: geometry collision mesh filename=package://rb1_base_description/meshes/wheels/wheel_rubber_6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; visual mesh filename=package://rb1_base_description/meshes/wheels/wheel_rubber_6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
- link rb1_omni_backwheel_link: geometry collision mesh filename=package://rb1_base_description/meshes/wheels/rb1v2_omniwhee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; visual mesh filename=package://rb1_base_description/meshes/wheels/rb1v2_omniwhee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
- link rb1_omni_front_leftwheel_link: geometry collision mesh filename=package://rb1_base_description/meshes/wheels/rb1v2_omniwhee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; visual mesh filename=package://rb1_base_description/meshes/wheels/rb1v2_omniwhee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
- link rb1_omni_front_rightwheel_link: geometry collision mesh filename=package://rb1_base_description/meshes/wheels/rb1v2_omniwhee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; visual mesh filename=package://rb1_base_description/meshes/wheels/rb1v2_omniwhee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
- link rb1_right_wheel_link: geometry collision mesh filename=package://rb1_base_description/meshes/wheels/wheel_rubber_6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; visual mesh filename=package://rb1_base_description/meshes/wheels/wheel_rubber_6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
- link rb1_torso_link: geometry collision mesh filename=package://rb1_base_description/meshes/others/adam_model.stl; visual mesh filename=package://rb1_base_description/meshes/others/rb1_torso_ur3.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
Joints:
- joint rb1_omni_front_leftwheel_joint: type fixed -> continuous
- joint rb1_omni_front_rightwheel_joint: type fixed -> continuous

Commit message: navigation to point added

File: paquetes_simulacion/rb1_base_description/robots/robotDummy.urdf (robot description, URDF)
Before this commit: robot rb1_base, 74 links, 73 joints
Links:
- link rb1_base_link: mass 100.0 -> 500.0
Joints:
- joint rb1_omni_backwheel_joint: type fixed -> continuous

Commit message: Accurate kinematics fixed

File: paquetes_simulacion/rb1_base_description/robots/robotDummy.urdf (robot description, URDF)
Before this commit: robot rb1_base, 74 links, 73 joints
Joints:
- joint rb1_omni_backwheel_joint: type fixed -> continuous

Commit message: ROS class in adam

File: paquetes_simulacion/rb1_base_description/robots/robotDummy.urdf (robot description, URDF)
Before this commit: robot rb1_base, 74 links, 73 joints
Links:
- added link rb1_torso_base_collision_link, mass 4.0; collision mesh filename=package://rb1_base_description/meshes/others/torso_base.stl; visual mesh filename=package://rb1_base_description/meshes/others/torso_base.stl
- added link rb1_torso_chest_collision_link, mass 4.0; collision mesh filename=package://rb1_base_description/meshes/others/torso_chest.stl; visual mesh filename=package://rb1_base_description/meshes/others/torso_chest.stl
- added link rb1_torso_shoulders_collision_link, mass 4.0; collision mesh filename=package://rb1_base_description/meshes/others/torso_shoulder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; visual mesh filename=package://rb1_base_description/meshes/others/torso_shoulder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
- link rb1_torso_link: geometry visual mesh filename=package://rb1_base_description/meshes/others/rb1_torso_ur3.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
Joints:
- added joint rb1_torso_base_collision_joint: type fixed, parent rb1_base_footprint, child rb1_torso_base_collision_link, origin xyz=-0.1 0.0 0.248 rpy=0.0 0.0 0.0, axis 0 0 1
- added joint rb1_torso_chest_collision_joint: type fixed, parent rb1_base_footprint, child rb1_torso_chest_collision_link, origin xyz=-0.1 0.0 0.248 rpy=0.0 0.0 0.0, axis 0 0 1
- added joint rb1_torso_shoulders_collision_joint: type fixed, parent rb1_base_footprint, child rb1_torso_shoulders_collision_link, origin xyz=-0.1 0.0 0.248 rpy=0.0 0.0 0.0, axis 0 0 1
