Commit message: Files structure updated

File: models/robot/rb1_base_description/robots/robotDummy.urdf (robot description, URDF)
Before this commit: robot rb1_base, 77 links, 76 joints
Joints:
- joint rb1_omni_backwheel_joint: origin xyz=-0.195 0.0 0.027 rpy=0 0 0 -> xyz=-0.195 0.0 0.026 rpy=0 0 0
- joint rb1_omni_front_leftwheel_joint: origin xyz=0.132 0.1535 0.027 rpy=0 0 0 -> xyz=0.132 0.1535 0.026 rpy=0 0 0
- joint rb1_omni_front_rightwheel_joint: origin xyz=0.132 -0.1535 0.027 rpy=0 0 0 -> xyz=0.132 -0.1535 0.026 rpy=0 0 0

Commit message: [PROBLEM SOLVED] Blocking Logic solved + DWA planner (not clean and not finished)

File: models/robot/rb1_base_description/robots/robotDummy.urdf (robot description, URDF)
Before this commit: robot rb1_base, 77 links, 76 joints
Links:
- link camera_link: mass None -> 0.0
- link joint_support_link: mass None -> 0.0
- link rgbd_link: mass None -> 0.0
- link shoulder_link: mass None -> 0.0
- link support_end_link: mass None -> 0.0
