Commit message: Grippers update and examples fixed

File: models/robot/rb1_base_description/robots/adam_grippers.urdf (robot description, URDF)
Before this commit: robot rb1_base, 77 links, 76 joints
Links:
- removed link L_dummy_link
- removed link L_hand_base_link
- removed link L_index_distal
- removed link L_index_proximal
- removed link L_middle_distal
- removed link L_middle_proximal
- removed link L_pinky_distal
- removed link L_pinky_proximal
- removed link L_ring_distal
- removed link L_ring_proximal
- removed link L_thumb_distal
- removed link L_thumb_intermediate
- removed link L_thumb_proximal
- removed link L_thumb_proximal_base
- removed link R_dummy_link
- removed link R_hand_base_link
- removed link R_index_distal
- removed link R_index_proximal
- removed link R_middle_distal
- removed link R_middle_proximal
- removed link R_pinky_distal
- removed link R_pinky_proximal
- removed link R_ring_distal
- removed link R_ring_proximal
- removed link R_thumb_distal
- removed link R_thumb_intermediate
- removed link R_thumb_proximal
- removed link R_thumb_proximal_base
- added link left_gripper_base_link, mass 6.165375582670241e-07; collision mesh filename=package://models/robot/grippers/meshes/base_link.stl scale=0.001 0.001 0.001; visual mesh filename=package://models/robot/grippers/meshes/base_link.stl scale=0.001 0.001 0.001
- added link left_gripper_chasis, mass 0.7358895650337893; visual mesh filename=package://models/robot/grippers/meshes/Chasis_Nuevo_v1_1_1_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 scale=0.001 0.001 0.001
- added link left_gripper_fsh-6w, mass 0.005462946868763102
- added link left_gripper_healical_gear, mass 0.06579799533400067; visual mesh filename=package://models/robot/grippers/meshes/Healical_Gear__6R@0.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 scale=0.001 0.001 0.001
- added link left_gripper_left_case, mass 0.10856430346764456; visual mesh filename=package://models/robot/grippers/meshes/Carcasa_v1_1.stl scale=0.001 0.001 0.001
- added link left_gripper_left_cover, mass 0.009556121937797202; collision mesh filename=package://models/robot/grippers/meshes/Cubrimiento_v1__1__1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 scale=0.001 0.001 0.001; visual mesh filename=package://models/robot/grippers/meshes/Cubrimiento_v1__1__1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 scale=0.001 0.001 0.001
- added link left_gripper_left_guia, mass 0.061978529347409946; visual mesh filename=package://models/robot/grippers/meshes/GuíaLeft_v1_1.stl scale=0.001 0.001 0.001
- added link left_gripper_left_paddle, mass 0.3072105701261476; visual mesh filename=package://models/robot/grippers/meshes/Conjunto_Herramienta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 scale=0.001 0.001 0.001
- added link left_gripper_left_pieza_movil, mass 0.026073243412509224; visual mesh filename=package://models/robot/grippers/meshes/PiezaMovilLeft_1.stl scale=0.001 0.001 0.001
- added link left_gripper_left_sensor, mass 0.007344505396044044
- added link left_gripper_left_zip, mass 0.1674750199260278; visual mesh filename=package://models/robot/grippers/meshes/CremalleraLeft_1.stl scale=0.001 0.001 0.001
- added link left_gripper_right_case, mass 0.10856430346765521; visual mesh filename=package://models/robot/grippers/meshes/Carcasa_v1__1__1_1_1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 scale=0.001 0.001 0.001
- added link left_gripper_right_cover, mass 0.009556048689960938; collision mesh filename=package://models/robot/grippers/meshes/Cubrimiento_v1_1_1_1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 scale=0.001 0.001 0.001; visual mesh filename=package://models/robot/grippers/meshes/Cubrimiento_v1_1_1_1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 scale=0.001 0.001 0.001
- added link left_gripper_right_guia, mass 0.061978529347409946; visual mesh filename=package://models/robot/grippers/meshes/GuíaRight_1.stl scale=0.001 0.001 0.001
- added link left_gripper_right_paddle, mass 0.30721057012614517; visual mesh filename=package://models/robot/grippers/meshes/Conjunto_Herramienta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 scale=0.001 0.001 0.001
- added link left_gripper_right_pieza_movil, mass 0.026073243412509224; visual mesh filename=package://models/robot/grippers/meshes/PiezaMovilRight_1.stl scale=0.001 0.001 0.001
- added link left_gripper_right_sensor, mass 0.007344505396044034
- added link left_gripper_right_zip, mass 0.1674750199260278; visual mesh filename=package://models/robot/grippers/meshes/CremalleraRight_v1_1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 scale=0.001 0.001 0.001
- added link left_gripper_servo, mass 0.027068171992842262
- added link left_gripper_tool0, mass 0.00
- added link right_gripper_base_link, mass 6.165375582670241e-07; visual mesh filename=package://models/robot/grippers/meshes/base_link.stl scale=0.001 0.001 0.001
- added link right_gripper_chasis, mass 0.7358895650337893; visual mesh filename=package://models/robot/grippers/meshes/Chasis_Nuevo_v1_1_1_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 scale=0.001 0.001 0.001
- added link right_gripper_fsh-6w, mass 0.005462946868763102
- added link right_gripper_healical_gear, mass 0.06579799533400067; visual mesh filename=package://models/robot/grippers/meshes/Healical_Gear__6R@0.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 scale=0.001 0.001 0.001
- added link right_gripper_left_case, mass 0.10856430346764456; visual mesh filename=package://models/robot/grippers/meshes/Carcasa_v1_1.stl scale=0.001 0.001 0.001
- added link right_gripper_left_cover, mass 0.009556121937797202; collision mesh filename=package://models/robot/grippers/meshes/Cubrimiento_v1__1__1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 scale=0.001 0.001 0.001; visual mesh filename=package://models/robot/grippers/meshes/Cubrimiento_v1__1__1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 scale=0.001 0.001 0.001
- added link right_gripper_left_guia, mass 0.061978529347409946; visual mesh filename=package://models/robot/grippers/meshes/GuíaLeft_v1_1.stl scale=0.001 0.001 0.001
- added link right_gripper_left_paddle, mass 0.3072105701261476; visual mesh filename=package://models/robot/grippers/meshes/Conjunto_Herramienta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 scale=0.001 0.001 0.001
- added link right_gripper_left_pieza_movil, mass 0.026073243412509224; visual mesh filename=package://models/robot/grippers/meshes/PiezaMovilLeft_1.stl scale=0.001 0.001 0.001
- added link right_gripper_left_sensor, mass 0.007344505396044044
- added link right_gripper_left_zip, mass 0.1674750199260278; visual mesh filename=package://models/robot/grippers/meshes/CremalleraLeft_1.stl scale=0.001 0.001 0.001
- added link right_gripper_right_case, mass 0.10856430346765521; visual mesh filename=package://models/robot/grippers/meshes/Carcasa_v1__1__1_1_1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 scale=0.001 0.001 0.001
- added link right_gripper_right_cover, mass 0.009556048689960938; collision mesh filename=package://models/robot/grippers/meshes/Cubrimiento_v1_1_1_1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 scale=0.001 0.001 0.001; visual mesh filename=package://models/robot/grippers/meshes/Cubrimiento_v1_1_1_1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 scale=0.001 0.001 0.001
- added link right_gripper_right_guia, mass 0.061978529347409946; visual mesh filename=package://models/robot/grippers/meshes/GuíaRight_1.stl scale=0.001 0.001 0.001
- added link right_gripper_right_paddle, mass 0.30721057012614517; visual mesh filename=package://models/robot/grippers/meshes/Conjunto_Herramienta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 scale=0.001 0.001 0.001
- added link right_gripper_right_pieza_movil, mass 0.026073243412509224; visual mesh filename=package://models/robot/grippers/meshes/PiezaMovilRight_1.stl scale=0.001 0.001 0.001
- added link right_gripper_right_sensor, mass 0.007344505396044034
- added link right_gripper_right_zip, mass 0.1674750199260278; visual mesh filename=package://models/robot/grippers/meshes/CremalleraRight_v1_1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 scale=0.001 0.001 0.001
- added link right_gripper_servo, mass 0.027068171992842262
- added link right_gripper_tool0, mass 0.00
- link camera_link: mass 0.0 -> None
- link joint_support_link: mass 0.0 -> None
- link rgbd_link: mass 0.0 -> None
- link shoulder_link: mass 0.0 -> None
- link support_end_link: mass 0.0 -> None
Joints:
- removed joint L_dummy_joint
- removed joint L_index_DIP_joint
- removed joint L_index_MCP_joint
- removed joint L_middle_DIP_joint
- removed joint L_middle_MCP_joint
- removed joint L_pinky_DIP_joint
- removed joint L_pinky_MCP_joint
- removed joint L_ring_DIP_joint
- removed joint L_ring_MCP_joint
- removed joint L_thumb_DIP_joint
- removed joint L_thumb_MCP_joint1
- removed joint L_thumb_MCP_joint2
- removed joint L_thumb_PIP_joint
- removed joint R_dummy_joint
- removed joint R_index_DIP_joint
- removed joint R_index_MCP_joint
- removed joint R_middle_DIP_joint
- removed joint R_middle_MCP_joint
- removed joint R_pinky_DIP_joint
- removed joint R_pinky_MCP_joint
- removed joint R_ring_DIP_joint
- removed joint R_ring_MCP_joint
- removed joint R_thumb_DIP_joint
- removed joint R_thumb_MCP_joint1
- removed joint R_thumb_MCP_joint2
- removed joint R_thumb_PIP_joint
- removed joint left_hand_base_joint
- removed joint right_hand_base_joint
- added joint left_gripper_LeftPaddle: type prismatic, parent left_gripper_left_guia, child left_gripper_left_pieza_movil, origin xyz=0.112068 0.000675 -0.016016 rpy=0 0 0, axis -0.0 -1.0 -0.0, limit lower=-0.035 upper=0.0 effort=100 velocity=100
- added joint left_gripper_RightPaddle: type prismatic, parent left_gripper_right_guia, child left_gripper_right_pieza_movil, origin xyz=-0.112068 0.000675 -0.014684 rpy=0 0 0, axis 0.0 -1.0 0.0, limit lower=0.0 upper=0.035 effort=100 velocity=100
- added joint left_gripper_Rigid 119: type fixed, parent left_gripper_chasis, child left_gripper_servo, origin xyz=0.005 -0.0148 0.053 rpy=0 0 0
- added joint left_gripper_Rigid 120: type fixed, parent left_gripper_servo, child left_gripper_fsh-6w, origin xyz=-0.004765 0.013919 0.014055 rpy=0 0 0
- added joint left_gripper_Rigid 121: type fixed, parent left_gripper_fsh-6w, child left_gripper_healical_gear, origin xyz=0.0075 0.0 0.00221 rpy=0 0 0
- added joint left_gripper_Rigid 122: type fixed, parent left_gripper_chasis, child left_gripper_left_case, origin xyz=0.0257 0.0 0.01 rpy=0 0 0
- added joint left_gripper_Rigid 123: type fixed, parent left_gripper_chasis, child left_gripper_right_case, origin xyz=-0.0257 0.0 0.01 rpy=0 0 0
- added joint left_gripper_Rigid 129: type fixed, parent left_gripper_right_paddle, child left_gripper_right_cover, origin xyz=0.0374 0.02005 0.069 rpy=0 0 0
- added joint left_gripper_Rigid 130: type fixed, parent left_gripper_right_paddle, child left_gripper_right_sensor, origin xyz=0.0374 0.02005 0.069 rpy=0 0 0
- added joint left_gripper_Rigid 131: type fixed, parent left_gripper_left_paddle, child left_gripper_left_sensor, origin xyz=-0.0374 -0.02005 0.069 rpy=0 0 0
- added joint left_gripper_Rigid 132: type fixed, parent left_gripper_right_pieza_movil, child left_gripper_right_zip, origin xyz=0.098818 0.009325 0.024934 rpy=0 0 0
- added joint left_gripper_Rigid 133: type fixed, parent left_gripper_left_pieza_movil, child left_gripper_left_zip, origin xyz=-0.098818 -0.010675 0.026266 rpy=0 0 0
- added joint left_gripper_Rigid 134: type fixed, parent left_gripper_left_zip, child left_gripper_left_paddle, origin xyz=0.0202 0.006926 0.012 rpy=0 0 0
- added joint left_gripper_Rigid 135: type fixed, parent left_gripper_right_zip, child left_gripper_right_paddle, origin xyz=-0.0202 -0.006925 0.012 rpy=0 0 0
- added joint left_gripper_Rigid 136: type fixed, parent left_gripper_left_paddle, child left_gripper_left_cover, origin xyz=-0.0374 -0.02005 0.069 rpy=0 0 0
- added joint left_gripper_RigidLeft: type fixed, parent left_gripper_chasis, child left_gripper_left_guia, origin xyz=0.00635 -0.04 0.09 rpy=0 0 0
- added joint left_gripper_RigidRight: type fixed, parent left_gripper_chasis, child left_gripper_right_guia, origin xyz=-0.00635 0.04 0.09 rpy=0 0 0
- added joint left_gripper_base_joint: type fixed, parent left_gripper_base_link, child left_gripper_tool0, origin xyz=0.0 0.0 0.159 rpy=0.0 0.0 0.0
- added joint left_gripper_base_link_to_body: type fixed, parent left_gripper_base_link, child left_gripper_chasis, origin xyz=0.000666 0.000675 0.0 rpy=0 0 0
- added joint rb1_left_arm_hand_joint: type fixed, parent rb1_left_arm_tool0, child left_gripper_base_link, origin xyz=0.0 0.0 0 rpy=0 0 0
- added joint rb1_right_arm_hand_joint: type fixed, parent rb1_right_arm_tool0, child right_gripper_base_link, origin xyz=0.0 0.0 0 rpy=0 0 0
- added joint right_gripper_LeftPaddle: type prismatic, parent right_gripper_left_guia, child right_gripper_left_pieza_movil, origin xyz=0.112068 0.000675 -0.016016 rpy=0 0 0, axis -0.0 -1.0 -0.0, limit lower=-0.035 upper=0.0 effort=100 velocity=100
- added joint right_gripper_RightPaddle: type prismatic, parent right_gripper_right_guia, child right_gripper_right_pieza_movil, origin xyz=-0.112068 0.000675 -0.014684 rpy=0 0 0, axis 0.0 -1.0 0.0, limit lower=0.0 upper=0.035 effort=100 velocity=100
- added joint right_gripper_Rigid 119: type fixed, parent right_gripper_chasis, child right_gripper_servo, origin xyz=0.005 -0.0148 0.053 rpy=0 0 0
- added joint right_gripper_Rigid 120: type fixed, parent right_gripper_servo, child right_gripper_fsh-6w, origin xyz=-0.004765 0.013919 0.014055 rpy=0 0 0
- added joint right_gripper_Rigid 121: type fixed, parent right_gripper_fsh-6w, child right_gripper_healical_gear, origin xyz=0.0075 0.0 0.00221 rpy=0 0 0
- added joint right_gripper_Rigid 122: type fixed, parent right_gripper_chasis, child right_gripper_left_case, origin xyz=0.0257 0.0 0.01 rpy=0 0 0
- added joint right_gripper_Rigid 123: type fixed, parent right_gripper_chasis, child right_gripper_right_case, origin xyz=-0.0257 0.0 0.01 rpy=0 0 0
- added joint right_gripper_Rigid 129: type fixed, parent right_gripper_right_paddle, child right_gripper_right_cover, origin xyz=0.0374 0.02005 0.069 rpy=0 0 0
- added joint right_gripper_Rigid 130: type fixed, parent right_gripper_right_paddle, child right_gripper_right_sensor, origin xyz=0.0374 0.02005 0.069 rpy=0 0 0
- added joint right_gripper_Rigid 131: type fixed, parent right_gripper_left_paddle, child right_gripper_left_sensor, origin xyz=-0.0374 -0.02005 0.069 rpy=0 0 0
- added joint right_gripper_Rigid 132: type fixed, parent right_gripper_right_pieza_movil, child right_gripper_right_zip, origin xyz=0.098818 0.009325 0.024934 rpy=0 0 0
- added joint right_gripper_Rigid 133: type fixed, parent right_gripper_left_pieza_movil, child right_gripper_left_zip, origin xyz=-0.098818 -0.010675 0.026266 rpy=0 0 0
- added joint right_gripper_Rigid 134: type fixed, parent right_gripper_left_zip, child right_gripper_left_paddle, origin xyz=0.0202 0.006926 0.012 rpy=0 0 0
- added joint right_gripper_Rigid 135: type fixed, parent right_gripper_right_zip, child right_gripper_right_paddle, origin xyz=-0.0202 -0.006925 0.012 rpy=0 0 0
- added joint right_gripper_Rigid 136: type fixed, parent right_gripper_left_paddle, child right_gripper_left_cover, origin xyz=-0.0374 -0.02005 0.069 rpy=0 0 0
- added joint right_gripper_RigidLeft: type fixed, parent right_gripper_chasis, child right_gripper_left_guia, origin xyz=0.00635 -0.04 0.09 rpy=0 0 0
- added joint right_gripper_RigidRight: type fixed, parent right_gripper_chasis, child right_gripper_right_guia, origin xyz=-0.00635 0.04 0.09 rpy=0 0 0
- added joint right_gripper_base_joint: type fixed, parent right_gripper_base_link, child right_gripper_tool0, origin xyz=0.0 0.0 0.159 rpy=0.0 0.0 0.0
- added joint right_gripper_base_link_to_body: type fixed, parent right_gripper_base_link, child right_gripper_chasis, origin xyz=0.000666 0.000675 0.0 rpy=0 0 0
